Commit message: Add files via upload

File: src/navigation/urdf/mybot.xacro (robot description, xacro)
@@ -19,5 +19,5 @@
     <collision name='collision'>
       <geometry>
-        <box size=".4 .2 .1"/>
+        <box size=".55 .386 .1"/>
       </geometry>
     </collision>
@@ -25,9 +25,9 @@
       <origin xyz="0 0 0.1" rpy=" 0 0 0"/>
       <geometry>
-        <box size=".4 .2 .1"/>
+        <box size=".55 .386 .1"/>
       </geometry>
     </visual>
     <collision name='caster_collision'>
-      <origin xyz="-0.15 0 0.05" rpy=" 0 0 0"/>
+      <origin xyz="0.14 0 0.05" rpy=" 0 0 0"/>
       <geometry>
         <sphere radius="0.05"/>
@@ -45,5 +45,5 @@
     </collision>
     <visual name='caster_visual'>
-      <origin xyz="-0.15 0 0.05" rpy=" 0 0 0"/>
+      <origin xyz="0.14 0 0.05" rpy=" 0 0 0"/>
       <geometry>
         <sphere radius="0.05"/>
@@ -51,5 +51,5 @@
     </visual>
     <collision name='caster_front_collision'>
-      <origin xyz="0.15 0 0.05" rpy=" 0 0 0"/>
+      <origin xyz="0.14 0 0.05" rpy=" 0 0 0"/>
       <geometry>
         <sphere radius="0.05"/>
@@ -67,5 +67,5 @@
     </collision>
     <visual name='caster_front_visual'>
-      <origin xyz="0.15 0 0.05" rpy=" 0 0 0"/>
+      <origin xyz="0.14 0 0.05" rpy=" 0 0 0"/>
       <geometry>
         <sphere radius="0.05"/>
@@ -76,13 +76,13 @@
     <!--origin xyz="0.1 0.13 0.1" rpy="0 1.5707 1.5707"/-->
     <collision name="collision">
-      <origin xyz="0 0 0.1" rpy="0 1.5707 1.5707"/>
-      <geometry>
-        <cylinder radius="0.1" length="0.05"/>
+      <origin xyz="-0.182 -0.211 0.075" rpy="0 1.5707 1.5707"/>
+      <geometry>
+        <cylinder radius="0.075" length="0.036"/>
       </geometry>
     </collision>
     <visual name="left_wheel_visual">
-      <origin xyz="0 0 0.1" rpy="0 1.5707 1.5707"/>
-      <geometry>
-        <cylinder radius="0.1" length="0.05"/>
+      <origin xyz="-0.182 -0.211 0.075" rpy="0 1.5707 1.5707"/>
+      <geometry>
+        <cylinder radius="0.075" length="0.036"/>
       </geometry>
     </visual>
@@ -99,13 +99,13 @@
     <!--origin xyz="0.1 -0.13 0.1" rpy="0 1.5707 1.5707"/-->
     <collision name="collision">
-      <origin xyz="0 0 0.1" rpy="0 1.5707 1.5707"/>
-      <geometry>
-        <cylinder radius="0.1" length="0.05"/>
+      <origin xyz="-0.182 0.211 0.075" rpy="0 1.5707 1.5707"/>
+      <geometry>
+        <cylinder radius="0.075" length="0.036"/>
       </geometry>
     </collision>
     <visual name="right_wheel_visual">
-      <origin xyz="0 0 0.1" rpy="0 1.5707 1.5707"/>
-      <geometry>
-        <cylinder radius="0.1" length="0.05"/>
+      <origin xyz="-0.182 0.211 0.075" rpy="0 1.5707 1.5707"/>
+      <geometry>
+        <cylinder radius="0.075" length="0.036"/>
       </geometry>
     </visual>
@@ -120,5 +120,5 @@
   </link>
   <joint type="continuous" name="left_wheel_hinge">
-    <origin xyz="0 0.15 0" rpy="0 0 0"/>
+    <origin xyz="-0.182 -0.193 0.075" rpy="0 0 0"/>
     <!--origin xyz="0.1 0.13 0" rpy="0 1.5707 1.5707"/-->
     <child link="left_wheel"/>
@@ -129,5 +129,5 @@
   </joint>
   <joint type="continuous" name="right_wheel_hinge">
-    <origin xyz="0 -0.15 0" rpy="0 0 0"/>
+    <origin xyz="-0.182 0.193 0.075" rpy="0 0 0"/>
     <!--origin xyz="0.1 -0.13 0" rpy="0 1.5707 1.5707"/-->
     <child link="right_wheel"/>
@@ -137,4 +137,5 @@
     <joint_properties damping="1.0" friction="1.0"/>
   </joint>
+<!--
   <link name="camera">
     <collision>
@@ -170,5 +171,4 @@
     <child link="laser"/>
   </joint>
-  <!-- Hokuyo Laser -->
   <link name="laser">
     <collision>
@@ -196,5 +196,4 @@
     <child link="imu_link"/>
   </joint>
-  <!-- Hokuyo Laser -->
   <link name="imu_link">
     <collision>
@@ -216,3 +215,4 @@
     </inertial>
   </link>
+-->
 </robot>

Commit message: urdf bot dimensions fixed

File: src/navigation/urdf/mybot.xacro (robot description, xacro)
@@ -76,5 +76,5 @@
     <!--origin xyz="0.1 0.13 0.1" rpy="0 1.5707 1.5707"/-->
     <collision name="collision">
-      <origin xyz="-0.182 -0.211 0.075" rpy="0 1.5707 1.5707"/>
+      <origin xyz="0 0 0" rpy="0 1.5707 1.5707"/>
       <geometry>
         <cylinder radius="0.075" length="0.036"/>
@@ -82,11 +82,11 @@
     </collision>
     <visual name="left_wheel_visual">
-      <origin xyz="-0.182 -0.211 0.075" rpy="0 1.5707 1.5707"/>
-      <geometry>
-        <cylinder radius="0.075" length="0.036"/>
-      </geometry>
-    </visual>
-    <inertial>
-      <origin xyz="0 0 0" rpy="0 1.5707 1.5707"/>
+      <origin xyz="0 0 0" rpy="0 1.5707 1.5707"/>
+      <geometry>
+        <cylinder radius="0.075" length="0.036"/>
+      </geometry>
+    </visual>
+    <inertial>
+      <origin xyz="0 0 0.1" rpy="0 1.5707 1.5707"/>
       <mass value="5"/>
       <inertia
@@ -99,5 +99,6 @@
     <!--origin xyz="0.1 -0.13 0.1" rpy="0 1.5707 1.5707"/-->
     <collision name="collision">
-      <origin xyz="-0.182 0.211 0.075" rpy="0 1.5707 1.5707"/>
+      <!--origin xyz="-0.182 0.211 0.075" rpy="0 1.5707 1.5707"/-->
+      <origin xyz="0 0 0" rpy="0 1.5707 1.5707"/>
       <geometry>
         <cylinder radius="0.075" length="0.036"/>
@@ -105,11 +106,11 @@
     </collision>
     <visual name="right_wheel_visual">
-      <origin xyz="-0.182 0.211 0.075" rpy="0 1.5707 1.5707"/>
-      <geometry>
-        <cylinder radius="0.075" length="0.036"/>
-      </geometry>
-    </visual>
-    <inertial>
-      <origin xyz="0 0 0" rpy="0 1.5707 1.5707"/>
+      <origin xyz="0 0 0" rpy="0 1.5707 1.5707"/>
+      <geometry>
+        <cylinder radius="0.075" length="0.036"/>
+      </geometry>
+    </visual>
+    <inertial>
+      <origin xyz="0 0 0.1" rpy="0 1.5707 1.5707"/>
       <mass value="5"/>
       <inertia
